File: hardware/usb2ax_v3.2.brd (EAGLE design)
At the start: 20 x 15 mm, 29 parts, among them Q1 CRYSTAL-0500290P1, U1 ATmega32u2, U2 IPC4282CZ6

Commit message: Upgraded to v3.2b : changed R3 from 150 to 47ohms for stronger line drive
Parts:
- R3: value 150R -> 47R
Other:
- board text added: "v3.2b"
- board text removed: "v3.2a"
Changed lines of the file:
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@@
 <?xml version="1.0" encoding="utf-8"?>
 <!DOCTYPE eagle SYSTEM "eagle.dtd">
-<eagle version="6.5.0">
+<eagle version="7.5.0">
 <drawing>
 <settings>
@@
 <layer number="19" name="Unrouted" color="6" fill="1" visible="yes" active="yes"/>
 <layer number="20" name="Dimension" color="15" fill="1" visible="yes" active="yes"/>
-<layer number="21" name="tPlace" color="7" fill="1" visible="yes" active="yes"/>
-<layer number="22" name="bPlace" color="7" fill="1" visible="no" active="yes"/>
-<layer number="23" name="tOrigins" color="15" fill="1" visible="yes" active="yes"/>
+<layer number="21" name="tPlace" color="7" fill="1" visible="no" active="yes"/>
+<layer number="22" name="bPlace" color="7" fill="1" visible="yes" active="yes"/>
+<layer number="23" name="tOrigins" color="15" fill="1" visible="no" active="yes"/>
 <layer number="24" name="bOrigins" color="15" fill="1" visible="no" active="yes"/>
 <layer number="25" name="tNames" color="7" fill="1" visible="no" active="yes"/>
@@
 <layer number="37" name="tTest" color="7" fill="1" visible="no" active="yes"/>
 <layer number="38" name="bTest" color="7" fill="1" visible="no" active="yes"/>
-<layer number="39" name="tKeepout" color="4" fill="11" visible="yes" active="yes"/>
+<layer number="39" name="tKeepout" color="4" fill="11" visible="no" active="yes"/>
 <layer number="40" name="bKeepout" color="1" fill="11" visible="no" active="yes"/>
 <layer number="41" name="tRestrict" color="4" fill="10" visible="no" active="yes"/>
@@
 <text x="10.95" y="12.85" size="0.7" layer="22" font="vector" ratio="17" rot="MR180">GND</text>
 <text x="7.61" y="1.16" size="2" layer="22" font="vector" ratio="17" rot="MR90">USB2AX</text>
-<text x="5.84" y="1.17" size="1.5" layer="22" font="vector" ratio="17" rot="MR90">v3.2a</text>
+<text x="5.84" y="1.17" size="1.5" layer="22" font="vector" ratio="17" rot="MR90">v3.2b</text>
 <text x="15.8" y="11.05" size="0.7" layer="22" font="vector" ratio="17" rot="MR90">GND</text>
 <text x="15.8" y="8.7" size="0.7" layer="22" font="vector" ratio="17" rot="MR90">12V</text>
@@
 <pass name="Default">
 <param name="RoutingGrid" value="50mil"/>
+<param name="AutoGrid" value="1"/>
+<param name="Efforts" value="0"/>
+<param name="TopRouterVariant" value="1"/>
 <param name="tpViaShape" value="round"/>
 <param name="PrefDir.1" value="|"/>
@@
 <element name="R1" library="Xevelabs" package="ARRAY_0402_65P_2_N" value="22R" x="7.1" y="6.42" rot="R225"/>
 <element name="R2" library="Xevelabs" package="ARRAY_0402_65P_2_N" value="150R" x="16.125" y="1.625" rot="R90"/>
-<element name="R3" library="Xevelabs" package="ARRAY_0402_65P_2_N" value="150R" x="13" y="2.4" rot="R90"/>
+<element name="R3" library="Xevelabs" package="ARRAY_0402_65P_2_N" value="47R" x="13" y="2.4" rot="R90"/>
 <element name="U2" library="Xevelabs" package="XSON6_N" value="IPC4282CZ6" x="6.08" y="7.65" rot="R135"/>
 <element name="USB1" library="Xevelabs" package="USB-A-THT" value="" x="2.7" y="7.5"/>
